Commit message: Edited the end effector

File: description/manipulator.control.xacro (robot description, xacro)
@@ -3,5 +3,5 @@
     <gazebo>
         <plugin filename="libgazebo_ros2_control.so" name="gazebo_ros2_control">
-            <parameters>$(find chess_manipulator)/config/controllers.yaml</parameters>
+            <parameters>$(find improves_chess)/config/controllers.yaml</parameters>
         </plugin>
     </gazebo>
@@ -12,6 +12,6 @@
         <joint name="panda_joint1">
             <command_interface name="position">
-                <param name="min">-2.8973</param>
-                <param name="max">2.8973</param>
+                <!-- <param name="min">-2.8973</param> -->
+                <!-- <param name="max">2.8973</param> -->
             </command_interface>
             <state_interface name="position" />
@@ -21,6 +21,6 @@
         <joint name="panda_joint2">
             <command_interface name="position">
-                <param name="min">-1.7628</param>
-                <param name="max">1.7628</param>
+                <!-- <param name="min">-1.7628</param> -->
+                <!-- <param name="max">1.7628</param> -->
             </command_interface>
             <state_interface name="position" />
@@ -30,6 +30,6 @@
         <joint name="panda_joint3">
             <command_interface name="position">
-                <param name="min">-2.8973</param>
-                <param name="max">2.8973</param>
+                <!-- <param name="min">-2.8973</param> -->
+                <!-- <param name="max">2.8973</param> -->
             </command_interface>
             <state_interface name="position" />
@@ -39,6 +39,6 @@
         <joint name="panda_joint4">
             <command_interface name="position">
-                <param name="min">-3.0718</param>
-                <param name="max">-0.0698</param>
+                <!-- <param name="min">-3.0718</param> -->
+                <!-- <param name="max">-0.0698</param> -->
             </command_interface>
             <state_interface name="position" />
@@ -48,6 +48,6 @@
         <joint name="panda_joint5">
             <command_interface name="position">
-                <param name="min">-2.8973</param>
-                <param name="max">2.8973</param>
+                <!-- <param name="min">-2.8973</param> -->
+                <!-- <param name="max">2.8973</param> -->
             </command_interface>
             <state_interface name="position" />
@@ -57,6 +57,6 @@
         <joint name="panda_joint6">
             <command_interface name="position">
-                <param name="min">-0.0175</param>
-                <param name="max">3.7525</param>
+                <!-- <param name="min">-0.0175</param> -->
+                <!-- <param name="max">3.7525</param> -->
             </command_interface>
             <state_interface name="position" />
@@ -66,15 +66,6 @@
         <joint name="panda_joint7">
             <command_interface name="position">
-                <param name="min">-2.8973</param>
-                <param name="max">2.8973</param>
-            </command_interface>
-            <state_interface name="position" />
-            <state_interface name="velocity" />
-            <state_interface name="effort" />
-        </joint>
-        <joint name="panda_joint8">
-            <command_interface name="position">
-                <param name="min">0</param>
-                <param name="max">0.1</param>
+                <!-- <param name="min">-0.0175</param> -->
+                <!-- <param name="max">3.7525</param> -->
             </command_interface>
             <state_interface name="position" />

File: description/manipulator.gazebo.xacro (robot description, xacro)
@@ -5,5 +5,5 @@
         <plugin name="gazebo_ros_joint_state_publisher"
             filename="libgazebo_ros_joint_state_publisher.so">
-            <update_rate>20</update_rate>
+            <update_rate>1000</update_rate>
             <joint_name>panda_joint1</joint_name>
             <joint_name>panda_joint2</joint_name>
@@ -13,7 +13,4 @@
             <joint_name>panda_joint6</joint_name>
             <joint_name>panda_joint7</joint_name>
-            <joint_name>panda_joint8</joint_name>
-            <joint_name>panda_finger_joint1</joint_name>
-            <joint_name>panda_finger_joint2</joint_name>
         </plugin>
     </gazebo>
@@ -21,11 +18,23 @@
     <!-- Friction parameters-->
     <gazebo reference="${robot_name}_link0">
-        <mu1>0.61</mu1>
-        <mu2>0.61</mu2>
+        <kp>0.0</kp>
+        <kd>0.0</kd>
+        <min_depth>0</min_depth>
+        <!-- <max_vel>0</max_vel> -->
+        <slip1>0</slip1>
+        <slip2>0</slip2>
+        <mu1>0</mu1>
+        <mu2>0</mu2>
     </gazebo>
     <!-- Link1 -->
     <gazebo reference="${robot_name}_link1">
-        <mu1>0.61</mu1>
-        <mu2>0.61</mu2>
+        <kp>0.0</kp>
+        <kd>0.0</kd>
+        <min_depth>0</min_depth>
+        <!-- <max_vel>0</max_vel> -->
+        <slip1>0</slip1>
+        <slip2>0</slip2>
+        <mu1>0</mu1>
+        <mu2>0</mu2>
     </gazebo>
     <!-- Link2 -->
@@ -51,31 +60,23 @@
     <!-- Link6 -->
     <gazebo reference="${robot_name}_link6">
-        <mu1>0.61</mu1>
-        <mu2>0.61</mu2>
+        <kp>100000.0</kp>
+        <kd>100.0</kd>
+        <min_depth>0</min_depth>
+        <!-- <max_vel>0</max_vel> -->
+        <slip1>0.2</slip1>
+        <slip2>0.2</slip2>
+        <mu>0.81</mu>
+        <mu2>0.5</mu2>
     </gazebo>
-    <!-- Link7 -->
     <gazebo reference="${robot_name}_link7">
-        <mu1>0.61</mu1>
-        <mu2>0.61</mu2>
-    </gazebo>
-    <!-- Link8 -->
-    <gazebo reference="${robot_name}_link8">
-        <mu1>0.61</mu1>
-        <mu2>0.61</mu2>
-    </gazebo>
-    <!-- LinkHand -->
-    <gazebo reference="${robot_name}_hand">
-        <mu1>0.61</mu1>
-        <mu2>0.61</mu2>
-    </gazebo>
-    <!-- LinkRightFinger -->
-    <gazebo reference="${robot_name}_rightfinger">
-        <mu1>0.61</mu1>
-        <mu2>0.61</mu2>
-    </gazebo>
-    <!-- LinkLeftFinger -->
-    <gazebo reference="${robot_name}_leftfinger">
-        <mu1>0.61</mu1>
-        <mu2>0.61</mu2>
+        <!-- <kp>50000.0</kp> -->
+        <kp>50000.0</kp>
+        <kd>1.0</kd>
+        <min_depth>0</min_depth>
+        <!-- <max_vel>0</max_vel> -->
+        <slip1>0</slip1>
+        <slip2>0</slip2>
+        <mu1>0</mu1>
+        <mu2>0</mu2>
     </gazebo>
 </robot>

File: description/manipulator.urdf.xacro (robot description, xacro)
@@ -4,9 +4,11 @@
   <link name="world" />
   <!-- Include arm and hand xacro files-->
-  <xacro:include filename="$(find chess_manipulator)/description/panda_arm.xacro" />
-  <xacro:include filename="$(find chess_manipulator)/description/panda_hand.xacro" />
+  <xacro:include filename="$(find improves_chess)/description/panda_arm.xacro" />
+  <xacro:include filename="$(find improves_chess)/description/panda_hand.xacro" />
   <!-- call the arm macro-->
   <xacro:panda_arm />
   <!-- call the hand macro-->
   <xacro:panda_hand ns="panda" rpy="0 0 ${-pi/4}" connected_to="panda_link8" />
+  <xacro:include filename="$(find improves_chess)/description/manipulator.gazebo.xacro" />
+  <xacro:include filename="$(find improves_chess)/description/manipulator.control.xacro" />
 </robot>

File: description/panda_arm.xacro (robot description, xacro)
@@ -42,5 +42,5 @@
   </xacro:macro>
   <xacro:macro name="panda_arm"
-    params="arm_id:='panda' description_pkg:='chess_manipulator' connected_to:='' xyz:='0 0 0' rpy:='0 0 0'">
+    params="arm_id:='panda' description_pkg:='improves_chess' connected_to:='' xyz:='0 0 0' rpy:='0 0 0'">
     <xacro:unless value="${not connected_to}">
       <joint name="${arm_id}_joint_${connected_to}" type="fixed">
@@ -61,10 +61,10 @@
       <visual>
         <geometry>
-          <mesh filename="file://$(find chess_manipulator)/meshes/visual/link0.dae" />
-        </geometry>
-      </visual>
-      <collision>
-        <geometry>
-          <mesh filename="file://$(find chess_manipulator)/meshes/collision/link0.stl" />
+          <mesh filename="file://$(find improves_chess)/meshes/visual/link0.dae" />
+        </geometry>
+      </visual>
+      <collision>
+        <geometry>
+          <mesh filename="file://$(find improves_chess)/meshes/collision/link0.stl" />
         </geometry>
       </collision>
@@ -75,13 +75,13 @@
       </inertial>
     </link>
-    --> <link name="${arm_id}_link1">
-      <visual>
-        <geometry>
-          <mesh filename="file://$(find chess_manipulator)/meshes/visual/link1.dae" />
-        </geometry>
-      </visual>
-      <collision>
-        <geometry>
-          <mesh filename="file://$(find chess_manipulator)/meshes/collision/link1.stl" />
+    <link name="${arm_id}_link1">
+      <visual>
+        <geometry>
+          <mesh filename="file://$(find improves_chess)/meshes/visual/link1.dae" />
+        </geometry>
+      </visual>
+      <collision>
+        <geometry>
+          <mesh filename="file://$(find improves_chess)/meshes/collision/link1.stl" />
         </geometry>
       </collision>
@@ -100,5 +100,6 @@
       <child link="${arm_id}_link1" />
       <axis xyz="0 0 1" />
-      <limit effort="87" lower="-2.8973" upper="2.8973" velocity="2.1750" />
+      <limit effort="87" lower="${-pi}" upper="${pi}" velocity="2.1750" />
+      <!-- <limit effort="87" lower="-2.8973" upper="2.8973" velocity="2.1750" /> -->
       <dynamics damping="${joint_damping}" />
     </joint>
@@ -106,10 +107,10 @@
       <visual>
         <geometry>
-          <mesh filename="file://$(find chess_manipulator)/meshes/visual/link2.dae" />
-        </geometry>
-      </visual>
-      <collision>
-        <geometry>
-          <mesh filename="file://$(find chess_manipulator)/meshes/collision/link2.stl" />
+          <mesh filename="file://$(find improves_chess)/meshes/visual/link2.dae" />
+        </geometry>
+      </visual>
+      <collision>
+        <geometry>
+          <mesh filename="file://$(find improves_chess)/meshes/collision/link2.stl" />
         </geometry>
       </collision>
@@ -128,5 +129,6 @@
       <child link="${arm_id}_link2" />
       <axis xyz="0 0 1" />
-      <limit effort="87" lower="-1.7628" upper="1.7628" velocity="2.1750" />
+      <limit effort="87" lower="${-pi}" upper="${pi}" velocity="2.1750" />
+      <!-- <limit effort="87" lower="-1.7628" upper="1.7628" velocity="2.1750" /> -->
       <dynamics damping="${joint_damping}" />
     </joint>
@@ -134,10 +136,10 @@
       <visual>
         <geometry>
-          <mesh filename="file://$(find chess_manipulator)/meshes/visual/link3.dae" />
-        </geometry>
-      </visual>
-      <collision>
-        <geometry>
-          <mesh filename="file://$(find chess_manipulator)/meshes/collision/link3.stl" />
+          <mesh filename="file://$(find improves_chess)/meshes/visual/link3.dae" />
+        </geometry>
+      </visual>
+      <collision>
+        <geometry>
+          <mesh filename="file://$(find improves_chess)/meshes/collision/link3.stl" />
         </geometry>
       </collision>
@@ -157,5 +159,6 @@
       <child link="${arm_id}_link3" />
       <axis xyz="0 0 1" />
-      <limit effort="87" lower="-2.8973" upper="2.8973" velocity="2.1750" />
+      <limit effort="87" lower="${-pi}" upper="${pi}" velocity="2.1750" />
+      <!-- <limit effort="87" lower="-2.8973" upper="2.8973" velocity="2.1750" /> -->
       <dynamics damping="${joint_damping}" />
     </joint>
@@ -163,10 +166,10 @@
       <visual>
         <geometry>
-          <mesh filename="file://$(find chess_manipulator)/meshes/visual/link4.dae" />
-        </geometry>
-      </visual>
-      <collision>
-        <geometry>
-          <mesh filename="file://$(find chess_manipulator)/meshes/collision/link4.stl" />
+          <mesh filename="file://$(find improves_chess)/meshes/visual/link4.dae" />
+        </geometry>
+      </visual>
+      <collision>
+        <geometry>
+          <mesh filename="file://$(find improves_chess)/meshes/collision/link4.stl" />
         </geometry>
       </collision>
@@ -186,5 +189,6 @@
       <child link="${arm_id}_link4" />
       <axis xyz="0 0 1" />
-      <limit effort="87" lower="-3.0718" upper="-0.0698" velocity="2.1750" />
+      <!-- <limit effort="87" lower="-3.0718" upper="-0.0698" velocity="2.1750" /> -->
+      <limit effort="87" lower="${-pi}" upper="${pi}" velocity="2.1750" />
       <dynamics damping="${joint_damping}" />
     </joint>
@@ -192,10 +196,10 @@
       <visual>
         <geometry>
-          <mesh filename="file://$(find chess_manipulator)/meshes/visual/link5.dae" />
-        </geometry>
-      </visual>
-      <collision>
-        <geometry>
-          <mesh filename="file://$(find chess_manipulator)/meshes/collision/link5.stl" />
+          <mesh filename="file://$(find improves_chess)/meshes/visual/link5.dae" />
+        </geometry>
+      </visual>
+      <collision>
+        <geometry>
+          <mesh filename="file://$(find improves_chess)/meshes/collision/link5.stl" />
         </geometry>
       </collision>
@@ -214,5 +218,6 @@
       <child link="${arm_id}_link5" />
       <axis xyz="0 0 1" />
-      <limit effort="12" lower="-2.8973" upper="2.8973" velocity="2.6100" />
+      <!-- <limit effort="12" lower="-2.8973" upper="2.8973" velocity="2.6100" /> -->
+      <limit effort="87" lower="${-pi}" upper="${pi}" velocity="2.1750" />
       <dynamics damping="${joint_damping}" />
     </joint>
@@ -220,10 +225,10 @@
       <visual>
         <geometry>
-          <mesh filename="file://$(find chess_manipulator)/meshes/visual/link6.dae" />
-        </geometry>
-      </visual>
-      <collision>
-        <geometry>
-          <mesh filename="file://$(find chess_manipulator)/meshes/collision/link6.stl" />
+          <mesh filename="file://$(find improves_chess)/meshes/visual/link6.dae" />
+        </geometry>
+      </visual>
+      <collision>
+        <geometry>
+          <mesh filename="file://$(find improves_chess)/meshes/collision/link6.stl" />
         </geometry>
       </collision>
@@ -242,5 +247,6 @@
       <child link="${arm_id}_link6" />
       <axis xyz="0 0 1" />
-      <limit effort="12" lower="-0.0175" upper="3.7525" velocity="2.6100" />
+      <!-- <limit effort="12" lower="-0.0175" upper="3.7525" velocity="2.6100" /> -->
+      <limit effort="87" lower="${-pi}" upper="${pi}" velocity="2.1750" />
       <dynamics damping="${joint_damping}" />
     </joint>
@@ -248,10 +254,10 @@
       <visual>
         <geometry>
-          <mesh filename="file://$(find chess_manipulator)/meshes/visual/link7.dae" />
-        </geometry>
-      </visual>
-      <collision>
-        <geometry>
-          <mesh filename="file://$(find chess_manipulator)/meshes/collision/link7.stl" />
+          <mesh filename="file://$(find improves_chess)/meshes/visual/link7.dae" />
+        </geometry>
+      </visual>
+      <collision>
+        <geometry>
+          <mesh filename="file://$(find improves_chess)/meshes/collision/link7.stl" />
         </geometry>
       </collision>
@@ -281,11 +287,11 @@
     </link>
     <joint
-      name="${arm_id}_joint8" type="revolute">
+      name="${arm_id}_joint8" type="fixed">
       <origin rpy="0 0 0" xyz="0 0 0.107" />
       <parent link="${arm_id}_link7" />
       <child link="${arm_id}_link8" />
-      <axis xyz="0 0 1" />
+      <!-- <axis xyz="0 0 1" />
       <limit effort="1" lower="0" upper="0.1" velocity="0.1" />
-      <dynamics damping="100" />
+      <dynamics damping="100" /> -->
     </joint>
   </xacro:macro>

File: description/panda_hand copy.xacro (robot description, xacro)
@@ -28,49 +28,49 @@
         <link name="${ns}_finger">
             <visual name='back'>
-                <origin xyz="-0.02 0 0.02" rpy="0 0 0" />
+                <origin xyz="0 0 0.025" rpy="0 0 0" />
                 <geometry>
-                    <box size="0.01 0.04 0.04" />
+                    <box size="0.02 0.08 0.05" />
                 </geometry>
             </visual>
             <visual name='left'>
-                <origin xyz="0 -0.02 0.02" rpy="0 0 0" />
+                <origin xyz="0.04 -0.04 0.03" rpy="0 0 0" />
                 <geometry>
-                    <box size="0.04 0.01 0.04" />
+                    <box size="0.08 0.02 0.04" />
                 </geometry>
             </visual>
             <visual name='right'>
-                <origin xyz="0 0.02 0.02" rpy="0 0 0" />
+                <origin xyz="0.04 0.04 0.03" rpy="0 0 0" />
                 <geometry>
-                    <box size="0.04 0.01 0.04" />
+                    <box size="0.08 0.02 0.04" />
                 </geometry>
             </visual>
             <visual name='front'>
-                <origin xyz="0.02 0 0.02" rpy="0 0 0" />
+                <origin xyz="0.08 0 0.025" rpy="0 0 0" />
                 <geometry>
-                    <box size="0.01 0.04 0.04" />
+                    <box size="0.02 0.08 0.05" />
                 </geometry>
             </visual>
             <collision name='back'>
-                <origin xyz="-0.02 0 0.02" rpy="0 0 0" />
+                <origin xyz="0 0 0.025" rpy="0 0 0" />
                 <geometry>
-                    <box size="0.01 0.04 0.04" />
+                    <box size="0.02 0.08 0.05" />
                 </geometry>
             </collision>
             <collision name='left'>
-                <origin xyz="0 -0.02 0.02" rpy="0 0 0" />
+                <origin xyz="0.04 -0.04 0.03" rpy="0 0 0" />
                 <geometry>
-                    <box size="0.04 0.01 0.04" />
+                    <box size="0.08 0.02 0.04" />
                 </geometry>
             </collision>
             <collision name='right'>
-                <origin xyz="0 0.02 0.02" rpy="0 0 0" />
+                <origin xyz="0.04 0.04 0.03" rpy="0 0 0" />
                 <geometry>
-                    <box size="0.04 0.01 0.04" />
+                    <box size="0.08 0.02 0.04" />
                 </geometry>
             </collision>
             <collision name='front'>
-                <origin xyz="0.02 0 0.02" rpy="0 0 0" />
+                <origin xyz="0.08 0 0.025" rpy="0 0 0" />
                 <geometry>
-                    <box size="0.01 0.04 0.04" />
+                    <box size="0.02 0.08 0.05" />
                 </geometry>
             </collision>
