Commit message: Fixed Bugs

File: description/manipulator.control.xacro (robot description, xacro)
@@ -3,5 +3,5 @@
     <gazebo>
         <plugin filename="libgazebo_ros2_control.so" name="gazebo_ros2_control">
-            <parameters>$(find improves_chess)/config/controllers.yaml</parameters>
+            <parameters>$(find chess_manipulator)/config/controllers.yaml</parameters>
         </plugin>
     </gazebo>

File: description/manipulator.urdf.xacro (robot description, xacro)
@@ -4,11 +4,11 @@
   <link name="world" />
   <!-- Include arm and hand xacro files-->
-  <xacro:include filename="$(find improves_chess)/description/panda_arm.xacro" />
-  <xacro:include filename="$(find improves_chess)/description/panda_hand.xacro" />
+  <xacro:include filename="$(find chess_manipulator)/description/panda_arm.xacro" />
+  <xacro:include filename="$(find chess_manipulator)/description/panda_hand.xacro" />
   <!-- call the arm macro-->
   <xacro:panda_arm />
   <!-- call the hand macro-->
   <xacro:panda_hand ns="panda" rpy="0 0 ${-pi/4}" connected_to="panda_link8" />
-  <xacro:include filename="$(find improves_chess)/description/manipulator.gazebo.xacro" />
-  <xacro:include filename="$(find improves_chess)/description/manipulator.control.xacro" />
+  <xacro:include filename="$(find chess_manipulator)/description/manipulator.gazebo.xacro" />
+  <xacro:include filename="$(find chess_manipulator)/description/manipulator.control.xacro" />
 </robot>

File: description/panda_arm.xacro (robot description, xacro)
@@ -42,5 +42,5 @@
   </xacro:macro>
   <xacro:macro name="panda_arm"
-    params="arm_id:='panda' description_pkg:='improves_chess' connected_to:='' xyz:='0 0 0' rpy:='0 0 0'">
+    params="arm_id:='panda' description_pkg:='chess_manipulator' connected_to:='' xyz:='0 0 0' rpy:='0 0 0'">
     <xacro:unless value="${not connected_to}">
       <joint name="${arm_id}_joint_${connected_to}" type="fixed">
@@ -61,10 +61,10 @@
       <visual>
         <geometry>
-          <mesh filename="file://$(find improves_chess)/meshes/visual/link0.dae" />
-        </geometry>
-      </visual>
-      <collision>
-        <geometry>
-          <mesh filename="file://$(find improves_chess)/meshes/collision/link0.stl" />
+          <mesh filename="file://$(find _chess)/meshes/visual/link0.dae" />
+        </geometry>
+      </visual>
+      <collision>
+        <geometry>
+          <mesh filename="file://$(find chess_manipulator)/meshes/collision/link0.stl" />
         </geometry>
       </collision>
@@ -78,10 +78,10 @@
       <visual>
         <geometry>
-          <mesh filename="file://$(find improves_chess)/meshes/visual/link1.dae" />
-        </geometry>
-      </visual>
-      <collision>
-        <geometry>
-          <mesh filename="file://$(find improves_chess)/meshes/collision/link1.stl" />
+          <mesh filename="file://$(find chess_manipulator)/meshes/visual/link1.dae" />
+        </geometry>
+      </visual>
+      <collision>
+        <geometry>
+          <mesh filename="file://$(find chess_manipulator)/meshes/collision/link1.stl" />
         </geometry>
       </collision>
@@ -107,10 +107,10 @@
       <visual>
         <geometry>
-          <mesh filename="file://$(find improves_chess)/meshes/visual/link2.dae" />
-        </geometry>
-      </visual>
-      <collision>
-        <geometry>
-          <mesh filename="file://$(find improves_chess)/meshes/collision/link2.stl" />
+          <mesh filename="file://$(find chess_manipulator)/meshes/visual/link2.dae" />
+        </geometry>
+      </visual>
+      <collision>
+        <geometry>
+          <mesh filename="file://$(find chess_manipulator)/meshes/collision/link2.stl" />
         </geometry>
       </collision>
@@ -136,10 +136,10 @@
       <visual>
         <geometry>
-          <mesh filename="file://$(find improves_chess)/meshes/visual/link3.dae" />
-        </geometry>
-      </visual>
-      <collision>
-        <geometry>
-          <mesh filename="file://$(find improves_chess)/meshes/collision/link3.stl" />
+          <mesh filename="file://$(find chess_manipulator)/meshes/visual/link3.dae" />
+        </geometry>
+      </visual>
+      <collision>
+        <geometry>
+          <mesh filename="file://$(find chess_manipulator)/meshes/collision/link3.stl" />
         </geometry>
       </collision>
@@ -166,10 +166,10 @@
       <visual>
         <geometry>
-          <mesh filename="file://$(find improves_chess)/meshes/visual/link4.dae" />
-        </geometry>
-      </visual>
-      <collision>
-        <geometry>
-          <mesh filename="file://$(find improves_chess)/meshes/collision/link4.stl" />
+          <mesh filename="file://$(find chess_manipulator)/meshes/visual/link4.dae" />
+        </geometry>
+      </visual>
+      <collision>
+        <geometry>
+          <mesh filename="file://$(find chess_manipulator)/meshes/collision/link4.stl" />
         </geometry>
       </collision>
@@ -196,10 +196,10 @@
       <visual>
         <geometry>
-          <mesh filename="file://$(find improves_chess)/meshes/visual/link5.dae" />
-        </geometry>
-      </visual>
-      <collision>
-        <geometry>
-          <mesh filename="file://$(find improves_chess)/meshes/collision/link5.stl" />
+          <mesh filename="file://$(find chess_manipulator)/meshes/visual/link5.dae" />
+        </geometry>
+      </visual>
+      <collision>
+        <geometry>
+          <mesh filename="file://$(find chess_manipulator)/meshes/collision/link5.stl" />
         </geometry>
       </collision>
@@ -225,10 +225,10 @@
       <visual>
         <geometry>
-          <mesh filename="file://$(find improves_chess)/meshes/visual/link6.dae" />
-        </geometry>
-      </visual>
-      <collision>
-        <geometry>
-          <mesh filename="file://$(find improves_chess)/meshes/collision/link6.stl" />
+          <mesh filename="file://$(find chess_manipulator)/meshes/visual/link6.dae" />
+        </geometry>
+      </visual>
+      <collision>
+        <geometry>
+          <mesh filename="file://$(find chess_manipulator)/meshes/collision/link6.stl" />
         </geometry>
       </collision>
@@ -254,10 +254,10 @@
       <visual>
         <geometry>
-          <mesh filename="file://$(find improves_chess)/meshes/visual/link7.dae" />
-        </geometry>
-      </visual>
-      <collision>
-        <geometry>
-          <mesh filename="file://$(find improves_chess)/meshes/collision/link7.stl" />
+          <mesh filename="file://$(find chess_manipulator)/meshes/visual/link7.dae" />
+        </geometry>
+      </visual>
+      <collision>
+        <geometry>
+          <mesh filename="file://$(find chess_manipulator)/meshes/collision/link7.stl" />
         </geometry>
       </collision>

File: description/panda_hand copy.xacro (robot description, xacro)
@@ -12,10 +12,10 @@
             <visual>
                 <geometry>
-                    <mesh filename="file://$(find improves_chess)/meshes/visual/hand.dae" />
+                    <mesh filename="file://$(find chess_manipulator)/meshes/visual/hand.dae" />
                 </geometry>
             </visual>
             <collision>
                 <geometry>
-                    <mesh filename="file://$(find improves_chess)/meshes/collision/hand.stl" />
+                    <mesh filename="file://$(find chess_manipulator)/meshes/collision/hand.stl" />
                 </geometry>
             </collision>

File: description/panda_hand.xacro (robot description, xacro)
@@ -12,10 +12,10 @@
             <visual>
                 <geometry>
-                    <mesh filename="file://$(find improves_chess)/meshes/visual/hand.dae" />
+                    <mesh filename="file://$(find chess_manipulator)/meshes/visual/hand.dae" />
                 </geometry>
             </visual>
             <collision>
                 <geometry>
-                    <mesh filename="file://$(find improves_chess)/meshes/collision/hand.stl" />
+                    <mesh filename="file://$(find chess_manipulator)/meshes/collision/hand.stl" />
                 </geometry>
             </collision>
