Commit message: Fixed Bugs

File: description/panda_arm.xacro (robot description, xacro)
@@ -61,5 +61,5 @@
       <visual>
         <geometry>
-          <mesh filename="file://$(find _chess)/meshes/visual/link0.dae" />
+          <mesh filename="file://$(find chess_manipulator)/meshes/visual/link0.dae" />
         </geometry>
       </visual>
